File: cat-ears-controller.kicad_pcb (KiCad board)
At the start: 2 copper layers, 70 x 29.5 mm, 21 parts, among them J1 Conn_01x04_MountingPin, J2 Conn_01x04_MountingPin, J3 Conn_01x02_MountingPin, J4 Conn_01x06, J5 Conn_01x02_MountingPin, SW1 SW_SPDT, SW2 SW_Push, SW3 SW_Push, SW4 SW_Push, SW5 SW_Push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

Commit message: Add servo connectors
Parts:
- added J6: Conn_01x03_MountingPin, Connector_JST:JST_ZH_B3B-ZR-SM4-TF_1x03-1MP_P1.50mm_Vertical, F.Cu at (75.5, 54.0)
- added J7: Conn_01x03_MountingPin, Connector_JST:JST_ZH_B3B-ZR-SM4-TF_1x03-1MP_P1.50mm_Vertical, F.Cu at (125.0, 54.0)
- moved D1 2.25 mm to (125.0, 47.8)
- moved D4 2.25 mm to (75.0, 47.8)
Connections:
- U1 pad 17: unconnected-(U1-P1.01_I2S_WS_D13-Pad17) -> /SERVO1
- U1 pad 21: unconnected-(U1-P1.03_SCK1_D17-Pad21) -> /SERVO2
Routing:
- net /SERVO2: track 0.00 -> 21.7 mm
- net /VBAT: track 157.2 -> 176.3 mm
- net /SERVO1: track 0.00 -> 17.8 mm
- net GND: track 11.7 -> 21.0 mm, vias 57 -> 70
- net Net-(J1-Pin_3): track 16.1 -> 18.6 mm
- net Net-(J2-Pin_4): track 17.1 -> 19.2 mm
- net Net-(J2-Pin_3): track 19.4 -> 21.5 mm
- net Net-(J3-Pin_1): track 68.6 -> 70.3 mm
- net Net-(D3-DOUT): track 12.5 -> 13.4 mm
- net /TXRX2: track 12.1 -> 13.0 mm
- net /WS2812: track 20.5 -> 21.1 mm
